Commit message: Added Kinova, updated UR5 xml

File: rocobench/envs/assets/kinova_with_base/base_with_kinova_gripper.urdf (robot description, URDF)
Before this commit: robot gen3_robotiq_2f_85, 22 links, 21 joints
Links:
- link left_inner_finger: geometry collision mesh filename=meshes/gripper/collision/robotiq_arg2f_85_inner_finger.stl scale=0.001 0.001 0.001; visual mesh filename=meshes/gripper/visual/robotiq_arg2f_85_inner_finger.stl scale=0.001 0.001 0.001
- link left_inner_finger_pad: geometry collision mesh filename=meshes/gripper/collision/robotiq_arg2f_85_pad.stl scale=0.001 0.001 0.001; visual mesh filename=meshes/gripper/visual/robotiq_arg2f_85_pad.stl scale=0.001 0.001 0.001
- link left_inner_knuckle: geometry collision mesh filename=meshes/gripper/collision/robotiq_arg2f_85_inner_knuckle.stl scale=0.001 0.001 0.001; visual mesh filename=meshes/gripper/visual/robotiq_arg2f_85_inner_knuckle.stl scale=0.001 0.001 0.001
- link left_outer_finger: geometry collision mesh filename=meshes/gripper/collision/robotiq_arg2f_85_outer_finger.stl scale=0.001 0.001 0.001; visual mesh filename=meshes/gripper/visual/robotiq_arg2f_85_outer_finger.stl scale=0.001 0.001 0.001
- link left_outer_knuckle: geometry collision mesh filename=meshes/gripper/collision/robotiq_arg2f_85_outer_knuckle.stl scale=0.001 0.001 0.001; visual mesh filename=meshes/gripper/visual/robotiq_arg2f_85_outer_knuckle.stl scale=0.001 0.001 0.001
- link right_inner_finger: geometry collision mesh filename=meshes/gripper/collision/robotiq_arg2f_85_inner_finger.stl scale=0.001 0.001 0.001; visual mesh filename=meshes/gripper/visual/robotiq_arg2f_85_inner_finger.stl scale=0.001 0.001 0.001
- link right_inner_finger_pad: geometry collision mesh filename=meshes/gripper/collision/robotiq_arg2f_85_pad.stl scale=0.001 0.001 0.001; visual mesh filename=meshes/gripper/visual/robotiq_arg2f_85_pad.stl scale=0.001 0.001 0.001
- link right_inner_knuckle: geometry collision mesh filename=meshes/gripper/collision/robotiq_arg2f_85_inner_knuckle.stl scale=0.001 0.001 0.001; visual mesh filename=meshes/gripper/visual/robotiq_arg2f_85_inner_knuckle.stl scale=0.001 0.001 0.001
- link right_outer_finger: geometry collision mesh filename=meshes/gripper/collision/robotiq_arg2f_85_outer_finger.stl scale=0.001 0.001 0.001; visual mesh filename=meshes/gripper/visual/robotiq_arg2f_85_outer_finger.stl scale=0.001 0.001 0.001
- link right_outer_knuckle: geometry collision mesh filename=meshes/gripper/collision/robotiq_arg2f_85_outer_knuckle.stl scale=0.001 0.001 0.001; visual mesh filename=meshes/gripper/visual/robotiq_arg2f_85_outer_knuckle.stl scale=0.001 0.001 0.001
